File: schematics/led_leveldriver/_saved_led_leveldriver.sch (KiCad schematic (older format))
At the start: 31 parts, among them IC1 TPIC6B595, J1 Conn_02x04_Odd_Even, J2 5V_IN, Q1 Q_PMOS_GSD, Q2 Q_PMOS_GSD, Q3 Q_PMOS_GSD, Q4 Q_PMOS_GSD, Q5 Q_PMOS_GSD, Q6 Q_PMOS_GSD, Q7 Q_PMOS_GSD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

Commit message: Rework Level driver to STM32 breakout board
Parts:
- added C6: 0.1uF, Capacitors_SMD:C_0603, symbol led_leveldriver-rescue:C
Connections:
- wire segments 168 -> 172
Changed lines of the file:
@@
 Wire Wire Line
 	1700 6450 1700 6250
+$Comp
+L led_leveldriver-rescue:C C6
+U 1 1 5B5EF735
+P 6000 2400
+F 0 "C6" H 6025 2500 50  0000 L CNN
+F 1 "0.1uF" H 6025 2300 50  0000 L CNN
+F 2 "Capacitors_SMD:C_0603" H 6038 2250 50  0001 C CNN
+F 3 "" H 6000 2400 50  0000 C CNN
+	1    6000 2400
+	1    0    0    -1
+$EndComp
+Wire Wire Line
+	5650 2150 6000 2150
+Wire Wire Line
+	6000 2150 6000 2250
+Wire Wire Line
+	5650 2600 6000 2600
+Wire Wire Line
+	6000 2600 6000 2550
 $EndSCHEMATC
