File: schematics/led_leveldriver/led_leveldriver.sch (KiCad schematic (older format))
At the start: 22 parts, among them IC1 TPIC6B595, J1 Conn_02x04_Odd_Even, Q1 Q_PMOS_GSD, Q2 Q_PMOS_GSD, Q3 Q_PMOS_GSD, Q4 Q_PMOS_GSD, Q5 Q_PMOS_GSD, Q6 Q_PMOS_GSD, Q7 Q_PMOS_GSD, Q8 Q_PMOS_GSD

Commit message: Rework Level driver to STM32 breakout board
Parts:
- removed BOARD_IN1: CONN_01X05, Pin_Headers:Pin_Header_Straight_1x05_Pitch2.54mm, symbol Conn_01x05
- added C1, C2: 10u, Capacitors_Tantalum_SMD:CP_Tantalum_Case-U_EIA-6032-15_Hand, symbol led_leveldriver-rescue:CP1
- added C3, C4, C?: 0.1uF, Capacitors_SMD:C_0603, symbol led_leveldriver-rescue:C
- added J2: 5V_IN, Connectors_Molex:Molex_MiniFit-JR-5556-02A_2x01x4.20mm_Straight, symbol Connector:Conn_01x02_Male
- added R1, R2: 10k, Resistors_SMD:R_0603, symbol led_leveldriver-rescue:R
- added U1: LM1117-3.3, TO_SOT_Packages_SMD:SOT-223-3_TabPin2, symbol led_leveldriver-rescue:LM1117-3.3
- added U2: BluePill_STM32F103C, BluePill_breakouts:BluePill_STM32F103C, symbol bluepill_breakouts:BluePill_STM32F103C
- added U3: 74HCT245, Housings_SOIC:SO-20_12.8x7.5mm_Pitch1.27mm, symbol 74hct245:74HCT245
- BOARD_OUT1: symbol Conn_01x05 -> led_leveldriver-rescue:Conn_01x05
- C5: renamed from C1; symbol C -> led_leveldriver-rescue:C
- IC1: symbol TPIC6B595 -> led_leveldriver-rescue:TPIC6B595
- J1: footprint Pin_Headers:Pin_Header_Angled_2x04_Pitch2.54mm -> Pin_Headers:Pin_Header_Straight_2x04_Pitch2.54mm; symbol Conn_02x04_Odd_Even -> led_leveldriver-rescue:Conn_02x04_Odd_Even
- Q1, Q2, Q3, Q4, Q5, Q6, Q7, Q8: symbol Q_PMOS_GSD -> led_leveldriver-rescue:Q_PMOS_GSD
- R10: renamed from R8; symbol R -> led_leveldriver-rescue:R
- R11: renamed from R9; symbol R -> led_leveldriver-rescue:R
- R3: renamed from R2; symbol R -> led_leveldriver-rescue:R
- R4: renamed from R3; symbol R -> led_leveldriver-rescue:R
- R5: renamed from R4; symbol R -> led_leveldriver-rescue:R
- R6: renamed from R5; symbol R -> led_leveldriver-rescue:R
- R7: renamed from R1; symbol R -> led_leveldriver-rescue:R
- R8: renamed from R6; symbol R -> led_leveldriver-rescue:R
- R9: renamed from R7; symbol R -> led_leveldriver-rescue:R
Connections:
- net labels added: +3V3, DATA, DOUT, L0, L1, L2, L3, L4, L5, L6, L7
- wire segments 104 -> 172
Other:
- moved on the sheet: BOARD_OUT1, C5, IC1, J1, Q1, Q2, Q3, Q4, Q5, Q6, Q7, Q8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
